File: hardware/PCB/TRV2_0.brd (EAGLE design)
At the start: 46 x 70 mm, 51 parts, among them IC1 TMP112, IC2 IC2, IC4 CNY70, IC5 ATMEGA8-AU, U1 DRV8850_RGY_24, X1 FC-12M

Commit message: before gerbers
Parts:
- moved R25 2.54 mm to (13.8, 61.5)
- moved J4 2.00 mm to (42.0, 21.0)
- moved U$2 1.51 mm to (13.2, 69.1)
- moved D5 1.46 mm to (13.1, 66.0)
Routing:
- net SPI_SCLK: track 41.1 -> 43.1 mm
- net SPI_MOSI: track 43.2 -> 45.2 mm
- net SPI_NNS: track 44.0 -> 46.0 mm
- net RFMIRQ: track 69.1 -> 71.0 mm
- net SPI_MISO: track 45.2 -> 47.1 mm
- net N$7: track 5.77 -> 7.38 mm
- net VCC: track 236.0 -> 234.5 mm
- net IO_POWER_UP: track 138.9 -> 138.0 mm, vias 5 -> 4
