File: hardware/PCB/TRV2_0.brd (EAGLE design)
At the start: 46 x 70 mm, 53 parts, among them IC1 TMP112, IC2 IC2, IC4 CNY70, IC5 ATMEGA8-AU, U1 DRV8850_RGY_24, X1 FC-12M

Commit message: More GND Via's added
Routing:
- net GND: vias 7 -> 53
Changed lines of the file:
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@@
 <setting verticaltext="up"/>
 </settings>
-<grid distance="0.003125" unitdist="mic" unit="mm" style="lines" multiple="1" display="no" altdistance="0.003125" altunitdist="mic" altunit="mm"/>
+<grid distance="0.05" unitdist="inch" unit="mm" style="lines" multiple="1" display="no" altdistance="0.003125" altunitdist="mic" altunit="mm"/>
 <layers>
 <layer number="1" name="Top" color="4" fill="1" visible="yes" active="yes"/>
@@
 <wire x1="46" y1="70" x2="0" y2="70" width="0" layer="20"/>
 <wire x1="0" y1="70" x2="0" y2="0" width="0" layer="20"/>
-<text x="6.0325" y="32.7025" size="0.8128" layer="25" rot="R180">IC2</text>
+<text x="1.480921875" y="35.26" size="0.8128" layer="25" rot="R270">IC2</text>
 <rectangle x1="12.76201875" y1="46.603265625" x2="13.55576875" y2="47.238265625" layer="1"/>
 <rectangle x1="12.76201875" y1="47.2458" x2="13.55576875" y2="47.8808" layer="1"/>
@@
 <elements>
 <element name="C1" library="rcl" package="C0603" value="100N" x="7.5184" y="34.3408" locked="yes" smashed="yes" rot="R270">
-<attribute name="NAME" x="8.7249" y="36.9443" size="0.8128" layer="25" rot="R180"/>
+<attribute name="NAME" x="8.477459375" y="37.0218" size="0.8128" layer="25" rot="R180"/>
 </element>
 <element name="C10" library="rcl" package="C0603" value="100N" x="18.0142125" y="21.202396875" locked="yes" smashed="yes">
@@
 </element>
 <element name="C17" library="rcl" package="C0603" value="0p" x="3.8608" y="15.8496" locked="yes" smashed="yes">
-<attribute name="NAME" x="2.9083" y="13.9446" size="0.8128" layer="25"/>
+<attribute name="NAME" x="1.936734375" y="14.9567375" size="0.8128" layer="25" rot="R90"/>
 </element>
 <element name="C2" library="rcl" package="C0603" value="100N" x="6.2992" y="38.8112" locked="yes" smashed="yes" rot="R270">
@@
 </element>
 <element name="IC5" library="Arduino-AVR" package="TQFP32-08" value="ATMEGA8-AU" x="10.26360625" y="21.649003125" locked="yes" smashed="yes">
-<attribute name="NAME" x="10.03500625" y="21.649003125" size="0.8128" layer="25"/>
+<attribute name="NAME" x="9.182378125" y="22.211815625" size="0.8128" layer="25"/>
 </element>
 <element name="J1" library="con-lstb" package="MA07-2" value="" x="20.4216" y="7.366" locked="yes" smashed="yes">
@@
 </element>
 <element name="R2" library="resistor" package="R0603" value="4K7" x="8.3312" y="12.5984" locked="yes" smashed="yes" rot="R270">
-<attribute name="NAME" x="7.7216" y="14.3637" size="0.8128" layer="25"/>
+<attribute name="NAME" x="7.0438875" y="12.0300375" size="0.8128" layer="25" rot="R90"/>
 </element>
 <element name="R21" library="resistor" package="R0603" value="47R" x="22.7584" y="43.0784" locked="yes" smashed="yes" rot="R90">
-<attribute name="NAME" x="23.9141" y="43.9166" size="0.8128" layer="25" rot="R270"/>
+<attribute name="NAME" x="20.684134375" y="44.063159375" size="0.8128" layer="25" rot="R270"/>
 </element>
 <element name="R22" library="resistor" package="R0603" value="1R0" x="18.0142125" y="17.951196875" locked="yes" smashed="yes" rot="R180">
@@
 <via x="18.415" y="34.29" extent="1-16" drill="0.6"/>
 <via x="14.605" y="28.321" extent="1-16" drill="0.6"/>
-<via x="29.845" y="5.461" extent="1-16" drill="0.6"/>
+<via x="30.335940625" y="5.334059375" extent="1-16" drill="0.6"/>
 <via x="3.81" y="32.385" extent="1-16" drill="0.6"/>
 <via x="10.795" y="38.735" extent="1-16" drill="0.6"/>
@@
 <wire x1="4.75120625" y1="38.2176" x2="6.2992" y2="38.2176" width="0.2032" layer="1"/>
 <wire x1="6.2992" y1="38.2176" x2="6.2992" y2="37.9612" width="0.4064" layer="1"/>
+<via x="35.7165625" y="60.92541875" extent="1-16" drill="0.6"/>
+<via x="35.797725" y="56.660765625" extent="1-16" drill="0.6"/>
+<via x="35.8203625" y="52.0790875" extent="1-16" drill="0.6"/>
+<via x="31.278121875" y="54.0701625" extent="1-16" drill="0.6"/>
+<via x="35.71200625" y="48.00714375" extent="1-16" drill="0.6"/>
+<via x="35.70523125" y="43.640371875" extent="1-16" drill="0.6"/>
+<via x="35.63750625" y="39.070153125" extent="1-16" drill="0.6"/>
+<via x="32.2379375" y="38.939884375" extent="1-16" drill="0.6"/>
+<via x="28.178821875" y="43.4631125" extent="1-16" drill="0.6"/>
+<via x="24.110271875" y="41.96135625" extent="1-16" drill="0.6"/>
+<via x="26.858509375" y="37.218353125" extent="1-16" drill="0.6"/>
+<via x="26.924534375" y="34.83234375" extent="1-16" drill="0.6"/>
+<via x="32.15085625" y="34.518953125" extent="1-16" drill="0.6"/>
+<via x="35.527440625" y="34.652621875" extent="1-16" drill="0.6"/>
+<via x="32.10755625" y="30.478253125" extent="1-16" drill="0.6"/>
+<via x="36.743740625" y="30.43901875" extent="1-16" drill="0.6"/>
+<via x="43.702059375" y="12.615459375" extent="1-16" drill="0.6"/>
+<wire x1="33.485203125" y1="10.060121875" x2="33.485203125" y2="10.060121875" width="0" layer="19" extent="1-16"/>
+<wire x1="37.329309375" y1="6.33808125" x2="37.329309375" y2="6.33808125" width="0" layer="19" extent="1-16"/>
+<via x="39.94780625" y="6.2553375" extent="1-16" drill="0.6"/>
+<via x="23.7337625" y="10.61684375" extent="1-16" drill="0.6"/>
+<via x="20.531971875" y="4.180421875" extent="1-16" drill="0.6"/>
+<via x="16.224159375" y="3.848103125" extent="1-16" drill="0.6"/>
+<via x="2.4530875" y="8.574228125" extent="1-16" drill="0.6"/>
+<via x="3.038271875" y="7.4826625" extent="1-16" drill="0.6"/>
+<via x="2.780709375" y="5.48315625" extent="1-16" drill="0.6"/>
+<via x="2.93293125" y="14.40289375" extent="1-16" drill="0.6"/>
+<via x="9.592915625" y="15.3272" extent="1-16" drill="0.6"/>
+<via x="8.52755625" y="14.876121875" extent="1-16" drill="0.6"/>
+<via x="8.094284375" y="22.0566875" extent="1-16" drill="0.6"/>
+<via x="8.66765625" y="23.882421875" extent="1-16" drill="0.6"/>
+<via x="14.554984375" y="25.91950625" extent="1-16" drill="0.6"/>
+<via x="12.64094375" y="22.530296875" extent="1-16" drill="0.6"/>
+<via x="19.546509375" y="23.08603125" extent="1-16" drill="0.6"/>
+<via x="5.1498625" y="29.906253125" extent="1-16" drill="0.6"/>
+<via x="4.108025" y="27.8471" extent="1-16" drill="0.6"/>
+<via x="4.97995" y="25.60586875" extent="1-16" drill="0.6"/>
+<via x="4.862903125" y="17.351821875" extent="1-16" drill="0.6"/>
+<via x="17.7169625" y="15.150215625" extent="1-16" drill="0.6"/>
+<via x="5.92226875" y="32.266821875" extent="1-16" drill="0.6"/>
+<via x="6.68294375" y="36.69413125" extent="1-16" drill="0.6"/>
+<wire x1="8.14590625" y1="39.875765625" x2="8.14590625" y2="39.875765625" width="0" layer="19" extent="1-16"/>
+<via x="18.902465625" y="41.336953125" extent="1-16" drill="0.6"/>
+<via x="8.865171875" y="36.511621875" extent="1-16" drill="0.6"/>
+<wire x1="9.63164375" y1="32.69780625" x2="9.63164375" y2="32.69780625" width="0" layer="19" extent="1-16"/>
+<via x="6.93210625" y="57.289828125" extent="1-16" drill="0.6"/>
+<via x="22.879778125" y="60.728040625" extent="1-16" drill="0.6"/>
+<via x="8.798390625" y="64.746703125" extent="1-16" drill="0.6"/>
+<via x="6.78496875" y="65.6578375" extent="1-16" drill="0.6"/>
+<via x="8.42350625" y="65.942903125" extent="1-16" drill="0.6"/>
 </signal>
 <signal name="SCL">
